File: AstroPix5/astropix_v5.kicad_pcb (KiCad board)
At the start: 4 copper layers, 56.4 x 65.6 mm, 39 parts, among them J1 HBOut, J12 Measures_Analog, J14 Bias, J2 Conn_01x05, J3 pcie_GECCO, J4 HBOut, J5 HBOut, J7 HV_in_external, J8 Conn_01x03, U2 AstroPix5_split_powerring

Commit message: Address PCB review comments: add stitching capacitors and increase track spacing
Parts:
- added C12: .1uF, Capacitor_SMD:C_0603_1608Metric, F.Cu at (181.3, 123.3)
- added C16: .1uF, Capacitor_SMD:C_0603_1608Metric, F.Cu at (196.1, 119.1)
- added C17: .1uF, Capacitor_SMD:C_0603_1608Metric, F.Cu at (183.8, 118.6)
- added C17: .1uF, Capacitor_SMD:C_0603_1608Metric, F.Cu at (194.7, 124.0)
- moved FID3 3.23 mm to (167.6, 69.3)
- moved C15 1.75 mm to (166.4, 87.5)
- moved R1 1.40 mm to (166.8, 84.3)
- moved C14 1.10 mm to (166.4, 91.5)
Routing:
- net GND: track 72.0 -> 82.6 mm, vias 10 -> 13
- net /SR_sin: track 42.0 -> 46.7 mm
- net Net-(J4-In): track 68.3 -> 64.1 mm
- net VDDA: track 26.8 -> 30.7 mm, vias 3 -> 6
- net /blpix: track 96.4 -> 100.2 mm
- net Net-(J14-Pin_10): track 63.7 -> 67.3 mm
- net Net-(U2A-Qdac<1>): track 30.4 -> 33.8 mm
- net Net-(J14-Pin_4): track 76.4 -> 73.1 mm
- net Net-(J14-Pin_12): track 61.5 -> 64.6 mm
- net /SR_ck2: track 42.8 -> 45.7 mm
- net Net-(JP4-B): track 44.7 -> 41.9 mm
- net /SPI_left_MISO0: track 43.3 -> 45.9 mm
- net /SR_ck1: track 40.6 -> 43.2 mm
- net /SPI_left_MISO1: track 44.9 -> 47.4 mm
- net Net-(J14-Pin_1): track 76.0 -> 78.5 mm
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