File: AstroPix5/astropix_v5_conn.kicad_sch (KiCad schematic)
At the start: 51 parts, among them J1 HBOut, J10 SPI_right, J12 Measures_Analog, J14 Bias, J2 Conn_01x05, J3 pcie_GECCO, J4 HBOut, J5 HBOut, J7 HV_in_external, J8 Conn_01x03, J9 SPI_left, U2 AstroPix5_split_powerring

Commit message: Fix ERC: remove duplicate SR_ck1/SR_ck2/SR_sin labels, fix duplicate PWR_FLAG, regenerate gerbers/PDF/pick-and-place
Parts:
- C11, C13, C4: MNP CC1210KKX7R8BB106 -> CC0603KRX5R6BB106
Connections:
- net SR_ck1: no longer J3.A42 (FMC_LA13_P)
- net SR_ck2: no longer J3.A43 (FMC_LA13_N)
- net SR_sin: no longer J3.B44 (FMC_LA12_P)
- no-connect marks 55 -> 58
